Commit message: Both arms display info now

File: so100.urdf (robot description, URDF)
Before this commit: robot so100, 7 links, 6 joints
Links:
- link base_link: geometry collision mesh filename=meshes/Base.STL scale=1 1 1; visual mesh filename=meshes/Base.STL scale=1 1 1
- link fixed_jaw_link: geometry collision mesh filename=meshes/Fixed_Jaw.STL scale=1 1 1; visual mesh filename=meshes/Fixed_Jaw.STL scale=1 1 1
- link forearm_link: geometry collision mesh filename=meshes/Forearm.STL scale=1 1 1; visual mesh filename=meshes/Forearm.STL scale=1 1 1
- link moving_jaw_link: geometry collision mesh filename=meshes/Moving_Jaw.STL scale=1 1 1; visual mesh filename=meshes/Moving_Jaw.STL scale=1 1 1
- link shoulder_link: geometry collision mesh filename=meshes/Shoulder_Rotation.STL scale=1 1 1; visual mesh filename=meshes/Shoulder_Rotation.STL scale=1 1 1
- link upper_arm_link: geometry collision mesh filename=meshes/Upper_Arm.STL scale=1 1 1; visual mesh filename=meshes/Upper_Arm.STL scale=1 1 1
- link wrist_link: geometry collision mesh filename=meshes/Wrist_Pitch_Roll.STL scale=1 1 1; visual mesh filename=meshes/Wrist_Pitch_Roll.STL scale=1 1 1
Joints:
- joint base_joint: origin xyz=0 0 0.0645 rpy=0 0 0 -> xyz=0 0 0.016 rpy=0 0 0
- joint forearm_joint: origin xyz=0 -0.11 0.004 rpy=0 0 0 -> xyz=0 -0.135 0.005 rpy=0 0 0
- joint shoulder_joint: origin xyz=0 0 0.062 rpy=0 0 0 -> xyz=0 -0.0305 0.1025 rpy=0 0 0
- joint upper_arm_joint: origin xyz=0 0.111 0.028 rpy=0 0 0 -> xyz=0 0.1125 0.028 rpy=0 0 0
